Commit message: First commit

File: sjtu_drone_description/urdf/sjtu_drone.urdf.xacro (robot description, xacro)
@@ -42,10 +42,10 @@
   </joint>
   <link name="sonar_link"/>
-  <joint name="front_cam_joint" type="fixed">
+  <joint name="depth_cam_joint" type="fixed">
     <origin rpy="0 0 0" xyz="0.2 0 0"/>
     <parent link="base_link" />
-    <child link="front_cam_link" />
-  </joint>
-  <link name="front_cam_link"/>
+    <child link="depth_cam_link" />
+  </joint>
+  <link name="depth_cam_link"/>
   <joint name="bottom_cam_joint" type="fixed">
     <origin rpy="0 ${M_PI/2} 0" xyz="0 0 0"/>
@@ -61,7 +61,7 @@
         <remapping>imu:=imu</remapping>
         <remapping>sonar:=sonar</remapping>
-        <remapping>camera_front:=camera_front</remapping>
+        <remapping>depth_front:=depth_front</remapping>
         <remapping>camera_bottom:=camera_bottom</remapping>
-        <remapping>camera_front_info:=camera_front_info</remapping>
+        <remapping>depth_front_info:=depth_front_info</remapping>
         <remapping>camera_bottom_info:=camera_bottom_info</remapping>
         <remapping>gps:=gps</remapping>
@@ -170,6 +170,6 @@
     </sensor>
   </gazebo>
-  <gazebo reference="front_cam_link">
-    <sensor name="front_camera" type="camera">
+  <gazebo reference="depth_cam_link">
+    <sensor name="depth_camera" type="depth">
       <always_on>1</always_on>
       <visualize>1</visualize>
@@ -180,5 +180,5 @@
           <width>640</width>
           <height>360</height>
-          <format>R8G8B8</format>
+          <format>B8G8R8</format>
         </image>
         <clip>
@@ -192,12 +192,14 @@
         </noise>
       </camera>
-      <plugin name="camera_front" filename="libgazebo_ros_camera.so">
-        <ros>
-          <namespace>${mp['namespace']}</namespace>
-          <!-- <remapping>~/image_raw:=camera_front</remapping>
-          <remapping>~/camera_info:=camera_front_info</remapping> -->
-        </ros>
-        <frame_name>${mp['namespace']}/front_cam_link</frame_name>
-        <camera_name>front</camera_name>
+      <plugin name="depth_front" filename="libgazebo_ros_camera.so">
+        <ros>
+          <namespace>${mp['namespace']}</namespace>
+          <!-- <remapping>~/image_raw:=depth_front</remapping>
+          <remapping>~/camera_info:=depth_front_info</remapping> -->
+        </ros>
+        <frame_name>${mp['namespace']}/depth_cam_link</frame_name>
+        <min_depth>0.1</min_depth>
+        <max_depth>100.0</max_depth>
+        <camera_name>depth</camera_name>
         <hack_baseline>0.07</hack_baseline>
       </plugin>
